File: pcb/bitski.kicad_pcb (KiCad board)
At the start: 2 copper layers, 83.1 x 34.1 mm, 314 parts, among them J1 Conn_02x12_Odd_Even, U1 ESP32-S3-MINI-1-N8, U2 BQ25185, U3 XC6206PxxxMR, U4 USBLC6-2SC6, U5 GXHT40AD, U6 BMP580, U7 IS31FL3731-QF, U8 IS31FL3731-QF

Commit message: updated project
Parts:
- removed the REF** at (157.0, 64.7)
- removed the REF** at (154.7, 88.5)
- removed the REF** at (132.8, 66.6)
- removed the REF** at (169.0, 62.6)
- removed the REF** at (135.3, 76.2)
- removed the REF** at (147.3, 74.1)
- removed the REF** at (144.9, 64.4)
- removed the REF** at (120.7, 78.5)
- removed the REF** at (123.2, 76.0)
- removed the REF** at (152.2, 64.5)
- removed the REF** at (176.3, 69.9)
- removed the REF** at (152.3, 86.0)
- removed the REF** at (127.9, 61.9)
- removed the REF** at (176.4, 89.0)
- removed the REF** at (152.2, 62.1)
- removed the REF** at (169.0, 67.4)
- removed the REF** at (123.2, 88.0)
- removed the REF** at (169.1, 88.9)
- removed the REF** at (142.5, 64.3)
- removed the REF** at (154.6, 71.8)
- removed the REF** at (140.1, 85.9)
- removed the REF** at (142.5, 66.7)
- removed the REF** at (174.0, 76.9)
- removed the REF** at (137.7, 76.3)
- removed the REF** at (149.7, 67.0)
- removed the REF** at (142.6, 76.2)
- removed the REF** at (161.8, 74.3)
- removed the REF** at (125.5, 71.4)
- removed the REF** at (120.6, 73.8)
- removed the REF** at (164.3, 86.3)
- removed the REF** at (125.6, 80.9)
- removed the REF** at (145.0, 78.7)
- removed the REF** at (161.8, 64.7)
- removed the REF** at (159.4, 81.5)
- removed the REF** at (135.2, 73.9)
- removed the REF** at (166.7, 76.8)
- removed the REF** at (161.8, 69.5)
- removed the REF** at (171.5, 69.7)
- removed the REF** at (176.3, 72.3)
- removed the REF** at (123.2, 83.2)
- removed the REF** at (154.7, 81.3)
- removed the REF** at (161.8, 67.1)
- removed the REF** at (149.7, 69.4)
- removed the REF** at (142.6, 88.2)
- removed the REF** at (176.3, 67.5)
- removed the REF** at (157.1, 79.0)
- removed the REF** at (125.6, 76.1)
- removed the REF** at (176.4, 77.0)
- removed the REF** at (159.4, 88.7)
- removed the REF** at (137.7, 85.9)
- removed the REF** at (161.8, 71.9)
- removed the REF** at (144.9, 66.8)
- removed the REF** at (130.3, 66.7)
- removed the REF** at (144.9, 62.0)
- removed the REF** at (164.2, 64.8)
- removed the REF** at (140.1, 76.3)
- removed the REF** at (157.1, 88.6)
- removed the REF** at (123.1, 73.7)
- removed the REF** at (135.3, 88.2)
- removed the REF** at (135.2, 71.5)
- removed the REF** at (132.9, 83.3)
- removed the REF** at (171.6, 84.0)
- removed the REF** at (149.8, 88.5)
- removed the REF** at (174.0, 86.5)
- removed the REF** at (176.3, 74.7)
- removed the REF** at (132.8, 61.8)
- removed the REF** at (173.9, 72.2)
- removed the REF** at (145.0, 76.3)
- removed the REF** at (171.6, 88.8)
- removed the REF** at (169.1, 86.5)
- removed the REF** at (130.4, 81.0)
- removed the REF** at (164.2, 69.6)
- removed the REF** at (154.7, 78.9)
- removed the REF** at (137.6, 74.0)
- removed the REF** at (176.3, 65.1)
- removed the REF** at (147.4, 78.8)
- removed the REF** at (176.4, 81.8)
- removed the REF** at (173.9, 62.6)
- removed the REF** at (164.3, 81.5)
- removed the REF** at (137.7, 88.3)
- removed the REF** at (159.3, 69.6)
- removed the REF** at (135.3, 83.4)
- removed the REF** at (132.9, 85.7)
- removed the REF** at (135.2, 66.7)
- removed the REF** at (157.1, 83.8)
- removed the REF** at (157.0, 62.3)
- removed the REF** at (135.2, 61.9)
- removed the REF** at (166.6, 72.1)
- removed the REF** at (169.0, 69.8)
- removed the REF** at (173.9, 67.4)
- removed the REF** at (140.0, 69.2)
- removed the REF** at (120.6, 69.0)
- removed the REF** at (140.0, 62.0)
- removed the REF** at (142.6, 83.4)
- removed the REF** at (166.6, 62.5)
- removed the REF** at (164.2, 62.4)
- removed the REF** at (171.6, 76.8)
- removed the REF** at (142.6, 81.0)
- removed the REF** at (147.4, 88.4)
- removed the REF** at (128.0, 78.6)
- removed the REF** at (130.4, 83.4)
- removed the REF** at (120.7, 76.1)
- removed the REF** at (171.5, 72.1)
- removed the REF** at (159.4, 76.7)
- removed the REF** at (161.9, 88.6)
- removed the REF** at (171.5, 67.3)
- removed the REF** at (140.0, 71.6)
- removed the REF** at (125.5, 61.8)
- removed the REF** at (159.4, 79.1)
- removed the REF** at (174.0, 81.7)
- removed the REF** at (176.4, 79.4)
- removed the REF** at (130.3, 64.3)
- removed the REF** at (169.1, 81.7)
- removed the REF** at (130.3, 71.5)
- removed the REF** at (149.8, 78.9)
- removed the REF** at (127.9, 71.5)
- removed the REF** at (145.0, 81.1)
- removed the REF** at (166.7, 84.0)
- removed the REF** at (174.0, 84.1)
- removed the REF** at (135.2, 69.1)
- removed the REF** at (154.6, 67.0)
- removed the REF** at (154.6, 62.2)
- removed the REF** at (149.7, 62.2)
- removed the REF** at (132.8, 71.4)
- removed the REF** at (137.7, 81.1)
- removed the REF** at (157.0, 69.5)
- removed the REF** at (159.3, 67.2)
- removed the REF** at (130.3, 61.9)
- removed the REF** at (147.4, 86.0)
- removed the REF** at (125.6, 88.1)
- removed the REF** at (176.3, 62.7)
- removed the REF** at (164.2, 74.4)
- removed the REF** at (123.1, 68.9)
- removed the REF** at (171.5, 62.5)
- removed the REF** at (140.0, 74.0)
- removed the REF** at (169.0, 74.6)
- removed the REF** at (173.9, 69.8)
- removed the REF** at (169.0, 65.0)
- removed the REF** at (142.5, 73.9)
- removed the REF** at (125.6, 78.5)
- removed the REF** at (166.6, 74.5)
- removed the REF** at (169.0, 72.2)
- removed the REF** at (132.8, 64.2)
- removed the REF** at (174.0, 79.3)
- removed the REF** at (147.4, 76.4)
- removed the REF** at (147.3, 64.5)
- removed the REF** at (127.9, 66.7)
- removed the REF** at (120.6, 61.8)
- removed the REF** at (142.5, 69.1)
- removed the REF** at (169.1, 79.3)
- removed the REF** at (171.5, 64.9)
- removed the REF** at (130.4, 88.2)
- removed the REF** at (123.2, 85.6)
- removed the REF** at (149.8, 81.3)
- removed the REF** at (174.0, 88.9)
- removed the REF** at (154.7, 76.5)
- removed the REF** at (135.3, 78.6)
- removed the REF** at (157.1, 76.6)
- removed the REF** at (161.9, 76.6)
- removed the REF** at (137.6, 66.8)
- removed the REF** at (149.7, 64.6)
- removed the REF** at (147.4, 83.6)
- removed the REF** at (132.9, 88.1)
- removed the REF** at (142.6, 78.6)
- removed the REF** at (149.8, 86.1)
- removed the REF** at (142.6, 85.8)
- removed the REF** at (171.5, 74.5)
- removed the REF** at (123.1, 61.7)
- removed the REF** at (164.3, 76.7)
- removed the REF** at (159.3, 72.0)
- removed the REF** at (135.2, 64.3)
- removed the REF** at (128.0, 83.4)
- removed the REF** at (157.0, 74.3)
- removed the REF** at (159.3, 62.4)
- removed the REF** at (135.3, 81.0)
- removed the REF** at (125.5, 64.2)
- removed the REF** at (157.1, 86.2)
- removed the REF** at (140.0, 64.4)
- removed the REF** at (137.7, 83.5)
- removed the REF** at (140.1, 81.1)
- removed the REF** at (132.8, 69.0)
- removed the REF** at (149.8, 83.7)
- removed the REF** at (142.5, 71.5)
- removed the REF** at (152.2, 71.7)
- removed the REF** at (147.3, 71.7)
- removed the REF** at (152.3, 76.4)
- removed the REF** at (161.9, 81.4)
- removed the REF** at (166.7, 88.8)
- removed the REF** at (152.3, 83.6)
- removed the REF** at (154.6, 69.4)
- removed the REF** at (137.6, 69.2)
- removed the REF** at (149.7, 74.2)
- removed the REF** at (173.9, 65.0)
- removed the REF** at (157.0, 71.9)
- removed the REF** at (176.4, 84.2)
- removed the REF** at (120.6, 64.2)
- removed the REF** at (166.6, 67.3)
- removed the REF** at (152.3, 78.8)
- removed the REF** at (128.0, 81.0)
- removed the REF** at (144.9, 71.6)
- removed the REF** at (152.3, 88.4)
- removed the REF** at (159.3, 74.4)
- removed the REF** at (130.4, 78.6)
- removed the REF** at (145.0, 83.5)
- removed the REF** at (125.5, 66.6)
- removed the REF** at (120.7, 88.1)
- removed the REF** at (132.9, 80.9)
- removed the REF** at (149.8, 76.5)
- removed the REF** at (132.8, 73.8)
- removed the REF** at (137.6, 71.6)
- removed the REF** at (145.0, 85.9)
- removed the REF** at (152.2, 69.3)
- removed the REF** at (161.9, 79.0)
- removed the REF** at (140.1, 83.5)
- removed the REF** at (169.1, 84.1)
- removed the REF** at (166.7, 86.4)
- removed the REF** at (171.6, 79.2)
- removed the REF** at (152.3, 81.2)
- removed the REF** at (154.7, 83.7)
- removed the REF** at (135.3, 85.8)
- removed the REF** at (157.0, 67.1)
- removed the REF** at (147.4, 81.2)
- removed the REF** at (144.9, 69.2)
- removed the REF** at (164.3, 83.9)
- removed the REF** at (125.6, 83.3)
- removed the REF** at (152.2, 66.9)
- removed the REF** at (123.1, 66.5)
- removed the REF** at (166.7, 81.6)
- removed the REF** at (159.4, 83.9)
- removed the REF** at (147.3, 66.9)
- removed the REF** at (127.9, 69.1)
- removed the REF** at (130.4, 76.2)
- removed the REF** at (154.6, 74.2)
- removed the REF** at (145.0, 88.3)
- removed the REF** at (171.6, 86.4)
- removed the REF** at (173.9, 74.6)
- removed the REF** at (120.7, 80.9)
- removed the REF** at (127.9, 73.9)
- removed the REF** at (157.1, 81.4)
- removed the REF** at (147.3, 69.3)
- removed the REF** at (128.0, 76.2)
- removed the REF** at (140.0, 66.8)
- removed the REF** at (123.2, 80.8)
- removed the REF** at (130.3, 73.9)
- removed the REF** at (120.7, 85.7)
- removed the REF** at (140.1, 88.3)
- removed the REF** at (159.3, 64.8)
- removed the REF** at (127.9, 64.3)
- removed the REF** at (164.3, 88.7)
- removed the REF** at (132.9, 76.1)
- removed the REF** at (140.1, 78.7)
- removed the REF** at (137.6, 62.0)
- removed the REF** at (149.7, 71.8)
- removed the REF** at (166.6, 69.7)
- removed the REF** at (164.3, 79.1)
- removed the REF** at (154.6, 64.6)
- removed the REF** at (120.6, 66.6)
- removed the REF** at (125.6, 85.7)
- removed the REF** at (130.4, 85.8)
- removed the REF** at (128.0, 88.2)
- removed the REF** at (152.2, 74.1)
- removed the REF** at (120.7, 83.3)
- removed the REF** at (164.2, 67.2)
- removed the REF** at (161.9, 86.2)
- removed the REF** at (147.3, 62.1)
- removed the REF** at (125.5, 69.0)
- removed the REF** at (123.1, 71.3)
- removed the REF** at (176.4, 86.6)
- removed the REF** at (130.3, 69.1)
- removed the REF** at (154.7, 86.1)
- removed the REF** at (137.6, 64.4)
- removed the REF** at (128.0, 85.8)
- removed the REF** at (123.2, 78.4)
- removed the REF** at (161.8, 62.3)
- removed the REF** at (144.9, 74.0)
- removed the REF** at (159.4, 86.3)
- removed the REF** at (125.5, 73.8)
- removed the REF** at (137.7, 78.7)
- removed the REF** at (166.6, 64.9)
- removed the REF** at (132.9, 78.5)
- removed the REF** at (120.6, 71.4)
- removed the REF** at (171.6, 81.6)
- removed the REF** at (123.1, 64.1)
- removed the REF** at (166.7, 79.2)
- removed the REF** at (161.9, 83.8)
- removed the REF** at (142.5, 61.9)
- removed the REF** at (164.2, 72.0)
- removed the REF** at (169.1, 76.9)
Routing:
- net (no net): track 3.72 -> 0.00 mm, vias 2 -> 0
