File: pcb/bitski.kicad_sch (KiCad schematic)
At the start: 40 parts, among them J1 Conn_02x12_Odd_Even, J2 USB_C_Receptacle_USB2.0_16P, J3 JST_XH_2.54mm, SW1 RESET, SW2 SW_Push_45deg, SW3 SW_Push_45deg, SW4 SW_Push_45deg, SW5 SW_Push_45deg, SW6 ON/OFF, U1 ESP32-S3-MINI-1-N8, U2 BQ25185, U3 XC6206PxxxMR, U4 USBLC6-2SC6, U5 GXHT40AD, U6 BMP580, U7 IS31FL3731-QF, U8 IS31FL3731-QF

Commit message: did so much omfg
Parts:
- removed C2: C_Small, Capacitor_SMD:C_0402_1005Metric, symbol Device:C_Small
- removed JP1: Jumper_2_Small_Bridged, symbol Jumper:Jumper_2_Small_Bridged
- added C11, C12: 22uF, symbol Device:C
- added D1: RED, symbol Device:LED
- added D7: ORANGE, symbol Device:LED
- added D8: GREEN, symbol Device:LED
- added JP1, JP2, JP3, JP4: (no value), symbol Jumper:SolderJumper_2_Open
- added R10, R8, R9: 1k, symbol Device:R
- added R11, R12: 10k, symbol Device:R
- added SW7: SW_Push, symbol Switch:SW_Push
- C10: value C_Small -> 0.1uF
- C9: value C_Small -> 10uF
- R1, R7: value 10k -> 4.7k
Connections:
- net +3V3: now also C10.1, U6.5 (SDO), U6.6 (CSB); no longer U8.2 (VCC)
- net +5V: now also D1.2 (A), D7.2 (A)
- net +BATT: now also C11.1
- net -BATT: now also C10.2, C11.2, C12.2, R10.2, R11.1, R12.2
- net BATT_LOAD: now also C12.1, D8.2 (A)
- net BMP580_SCL: now also JP1.1 (A)
- net BMP580_SDA: now also U6.4 (SDI), JP3.1 (A); no longer U6.5 (SDO)
- net SHT40_SCL: now also JP2.1 (A); no longer R1.2, U1.11 (IO7)
- net SHT40_SDA: now also JP4.1 (A); no longer R7.2, U1.10 (IO6)
- net SCL2: now reaches U1.12 (IO8)
- net SDA2: now reaches U1.13 (IO9)
- net GPIO0: now reaches U1.4 (IO0)
- net at U2.3 (STAT2): now also R9.2
- net at U2.4 (~{CE}): now also R11.2
- net at U2.6 (TS/MR): now also R12.1
- net VSET: now reaches U2.7 (VSET)
- net ISET: now reaches U2.8 (ISET)
- net at U2.9 (STAT1): now also R8.2
- new net: D1.1 (K), R8.1
- new net: D8.1 (K), R10.1
- new net: D7.1 (K), R9.1
- new net SCL1: JP1.2 (B), JP2.2 (B), R1.2, U1.10 (IO6)
- new net SDA1: JP3.2 (B), JP4.2 (B), R7.2, U1.11 (IO7)
Other:
- note added: "BMP 580! primarily measures barometric pressure, but can also +-0.5C on temp"
- note added: "Config block"
- note added: "Device has power"
- note added: "Items: - BMP580 - Battery voltages"
- note added: "POWER REG // THIS WILL NOT WORK"
- note added: "configured for i2c"
- note added: "i2c block"
- note added: "i2c, 0x47 7-bit"
- note added: "jumpers to test"
- note removed: "Power regulation"
- note removed: "need to change to bmp580 (check datasheet) primarily measures barometric pressure, but can also +-0.5C on temp"
- moved on the sheet: C1, C3, C7, C8, C9, J3, R4, R5, R6, SW1, U1, U2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

Commit message: updated project
Parts:
- removed D3: LED_45deg, Resistor_SMD:R_0402_1005Metric_Pad0.72x0.64mm_HandSolder, symbol Device:LED_45deg
- removed D4, D5, D6: LED_45deg, LED_SMD:LED_0402_1005Metric, symbol Device:LED_45deg
- added D10, D100, D101, D102, D103, D104, D105, D106, D107, D108, D109, D11, D110, D111, D112, D113, D114, D115, D116, D117, D118, D119, D12, D120, D121, D122, D123, D124, D125, D126, D127, D128, D129, D13, D130, D131, D132, D133, D134, D135, D136, D137, D138, D139, D14, D140, D141, D142, D143, D144, D145, D146, D147, D148, D15, D16, D17, D18, D19, D20, D21, D22, D23, D24, D25, D26, D27, D28, D29, D30, D31, D32, D33, D34, D35, D36, D37, D38, D39, D40, D41, D42, D43, D44, D45, D46, D47, D48, D49, D5, D50, D51, D52, D53, D54, D55, D56, D57, D58, D59, D6, D60, D61, D62, D63, D64, D65, D66, D67, D68, D69, D7, D70, D71, D72, D73, D74, D75, D76, D77, D78, D79, D8, D80, D81, D82, D83, D84, D85, D86, D87, D88, D89, D9, D90, D91, D92, D93, D94, D95, D96, D97, D98, D99: LED_Small, symbol Device:LED_Small
- added R13: 20k, symbol Device:R_Small
- renumbered D8 to D3, D7 to D4
Connections:
- net -BATT: now also U7.29 (GND), U7.5 (GND), U8.29 (GND), U8.5 (GND)
- net LED_SDA2: now reaches U8.19 (SDA)
- net POWER_LEDMATRIX: now reaches U8.2 (VCC)
- net POWER_LEDMATRIX: now also U7.2 (VCC)
- net LED_SCL2: now reaches U8.20 (SCL)
- net LED_SDA1: now reaches U7.19 (SDA)
- net LED_SCL1: now reaches U7.20 (SCL)
- net +5V renamed VUSB_CLEAN
- new net CA1: D10.1 (K), D11.1 (K), D12.1 (K), D13.2 (A), D21.2 (A), D29.2 (A), D37.2 (A), D45.2 (A), D5.1 (K), D53.2 (A), D6.1 (K), D61.2 (A), D69.2 (A), D7.1 (K), D8.1 (K), D9.1 (K)
- new net CA2: D13.1 (K), D14.1 (K), D15.1 (K), D16.1 (K), D17.1 (K), D18.1 (K), D19.1 (K), D20.1 (K), D22.2 (A), D30.2 (A), D38.2 (A), D46.2 (A), D5.2 (A), D54.2 (A), D62.2 (A), D70.2 (A)
- new net CA3: D14.2 (A), D21.1 (K), D22.1 (K), D23.1 (K), D24.1 (K), D25.1 (K), D26.1 (K), D27.1 (K), D28.1 (K), D31.2 (A), D39.2 (A), D47.2 (A), D55.2 (A), D6.2 (A), D63.2 (A), D71.2 (A)
- new net CA4: D15.2 (A), D23.2 (A), D29.1 (K), D30.1 (K), D31.1 (K), D32.1 (K), D33.1 (K), D34.1 (K), D35.1 (K), D36.1 (K), D40.2 (A), D48.2 (A), D56.2 (A), D64.2 (A), D7.2 (A), D72.2 (A)
- new net CA5: D16.2 (A), D24.2 (A), D32.2 (A), D37.1 (K), D38.1 (K), D39.1 (K), D40.1 (K), D41.1 (K), D42.1 (K), D43.1 (K), D44.1 (K), D49.2 (A), D57.2 (A), D65.2 (A), D73.2 (A), D8.2 (A)
- new net CA6: D17.2 (A), D25.2 (A), D33.2 (A), D41.2 (A), D45.1 (K), D46.1 (K), D47.1 (K), D48.1 (K), D49.1 (K), D50.1 (K), D51.1 (K), D52.1 (K), D58.2 (A), D66.2 (A), D74.2 (A), D9.2 (A)
- new net CA7: D10.2 (A), D18.2 (A), D26.2 (A), D34.2 (A), D42.2 (A), D50.2 (A), D53.1 (K), D54.1 (K), D55.1 (K), D56.1 (K), D57.1 (K), D58.1 (K), D59.1 (K), D60.1 (K), D67.2 (A), D75.2 (A)
- new net CA8: D11.2 (A), D19.2 (A), D27.2 (A), D35.2 (A), D43.2 (A), D51.2 (A), D59.2 (A), D61.1 (K), D62.1 (K), D63.1 (K), D64.1 (K), D65.1 (K), D66.1 (K), D67.1 (K), D68.1 (K), D76.2 (A)
- new net CA9: D12.2 (A), D20.2 (A), D28.2 (A), D36.2 (A), D44.2 (A), D52.2 (A), D60.2 (A), D68.2 (A), D69.1 (K), D70.1 (K), D71.1 (K), D72.1 (K), D73.1 (K), D74.1 (K), D75.1 (K), D76.1 (K)
- new net CB1: D104.1 (K), D113.1 (K), D122.1 (K), D131.1 (K), D140.1 (K), D77.1 (K), D78.2 (A), D79.2 (A), D80.2 (A), D81.2 (A), D82.2 (A), D83.2 (A), D84.2 (A), D85.2 (A), D86.1 (K), D95.1 (K)
- new net CB2: D105.1 (K), D114.1 (K), D123.1 (K), D132.1 (K), D141.1 (K), D77.2 (A), D78.1 (K), D87.1 (K), D88.2 (A), D89.2 (A), D90.2 (A), D91.2 (A), D92.2 (A), D93.2 (A), D94.2 (A), D96.1 (K)
- new net CB3: D100.2 (A), D101.2 (A), D102.2 (A), D103.2 (A), D106.1 (K), D115.1 (K), D124.1 (K), D133.1 (K), D142.1 (K), D79.1 (K), D86.2 (A), D87.2 (A), D88.1 (K), D97.1 (K), D98.2 (A), D99.2 (A)
- new net CB4: D107.1 (K), D108.2 (A), D109.2 (A), D110.2 (A), D111.2 (A), D112.2 (A), D116.1 (K), D125.1 (K), D134.1 (K), D143.1 (K), D80.1 (K), D89.1 (K), D95.2 (A), D96.2 (A), D97.2 (A), D98.1 (K)
- new net CB5: D104.2 (A), D105.2 (A), D106.2 (A), D107.2 (A), D108.1 (K), D117.1 (K), D118.2 (A), D119.2 (A), D120.2 (A), D121.2 (A), D126.1 (K), D135.1 (K), D144.1 (K), D81.1 (K), D90.1 (K), D99.1 (K)
- new net CB6: D100.1 (K), D109.1 (K), D113.2 (A), D114.2 (A), D115.2 (A), D116.2 (A), D117.2 (A), D118.1 (K), D127.1 (K), D128.2 (A), D129.2 (A), D130.2 (A), D136.1 (K), D145.1 (K), D82.1 (K), D91.1 (K)
- new net CB7: D101.1 (K), D110.1 (K), D119.1 (K), D122.2 (A), D123.2 (A), D124.2 (A), D125.2 (A), D126.2 (A), D127.2 (A), D128.1 (K), D137.1 (K), D138.2 (A), D139.2 (A), D146.1 (K), D83.1 (K), D92.1 (K)
- new net CB8: D102.1 (K), D111.1 (K), D120.1 (K), D129.1 (K), D131.2 (A), D132.2 (A), D133.2 (A), D134.2 (A), D135.2 (A), D136.2 (A), D137.2 (A), D138.1 (K), D147.1 (K), D148.2 (A), D84.1 (K), D93.1 (K)
- new net CB9: D103.1 (K), D112.1 (K), D121.1 (K), D130.1 (K), D139.1 (K), D140.2 (A), D141.2 (A), D142.2 (A), D143.2 (A), D144.2 (A), D145.2 (A), D146.2 (A), D147.2 (A), D148.1 (K), D85.1 (K), D94.1 (K)
Other:
- note added: "3v3 power reg"
- note added: "TODO: ADD TESTPOINTS EVERYWHERE! Polish step, has least # of dependencies"
- note added: "each IC supports 144 LEDs"
- note added: "selects i2c, address 0x47 7-bit"
- note removed: "LED Grid, 12x24 0603"
- note removed: "POWER REG // THIS WILL NOT WORK"
- note removed: "TODO: ADD TESTPOINTS EVERYWHERE"
- note removed: "TODO: add an LED here at the end, after generating the matrix"
- note removed: "double to support everything!"
- note removed: "i2c, 0x47 7-bit"
- moved on the sheet: J1, U7, U8
